Commit message: Updated moveit configs and placed packages in curie_ws

File: curie_ws/src/curie_arm_moveit_config/config/arm.urdf.xacro (robot description, xacro)
@@ -3,5 +3,5 @@
     <xacro:arg name="initial_positions_file" default="initial_positions.yaml" />
     <!-- Import arm urdf file -->
-    <xacro:include filename="$(find arm_visualizer)/urdf/arm.urdf" />
+    <xacro:include filename="$(find curie_robot_description)/urdf/arm.urdf" />
     <!-- Import control_xacro -->
     <xacro:include filename="arm.ros2_control.xacro" />

File: curie_ws/src/curie_robot_description/urdf/arm.urdf (robot description, URDF)
Before this commit: robot arm, 7 links, 6 joints
Links:
- link Baseplate_Part: geometry collision mesh filename=package://curie_robot_description/meshes/Baseplate_Part.STL; visual mesh filename=package://curie_robot_description/meshes/Baseplate_Part.STL
- link Bicep_Linkage: geometry collision mesh filename=package://curie_robot_description/meshes/Bicep_Linkage.STL; visual mesh filename=package://curie_robot_description/meshes/Bicep_Linkage.STL
- link Forearm_Linkage: geometry collision mesh filename=package://curie_robot_description/meshes/Forearm_Linkage.STL; visual mesh filename=package://curie_robot_description/meshes/Forearm_Linkage.STL
- link Shoulder: geometry collision mesh filename=package://curie_robot_description/meshes/Shoulder.STL; visual mesh filename=package://curie_robot_description/meshes/Shoulder.STL
- link Wrist_Pitch: geometry collision mesh filename=package://curie_robot_description/meshes/Wrist_Pitch.STL; visual mesh filename=package://curie_robot_description/meshes/Wrist_Pitch.STL
- link Wrist_Roll: geometry collision mesh filename=package://curie_robot_description/meshes/Wrist_Roll.STL; visual mesh filename=package://curie_robot_description/meshes/Wrist_Roll.STL

Commit message: Moved robot description for arm

File: curie_ws/src/curie_arm_moveit_config/config/arm.urdf.xacro (robot description, xacro)
@@ -3,5 +3,5 @@
     <xacro:arg name="initial_positions_file" default="initial_positions.yaml" />
     <!-- Import arm urdf file -->
-    <xacro:include filename="$(find curie_robot_description)/urdf/arm.urdf" />
+    <xacro:include filename="$(find curie_robot_description)/arm/urdf/arm.urdf" />
     <!-- Import control_xacro -->
     <xacro:include filename="arm.ros2_control.xacro" />

File: curie_ws/src/curie_robot_description/arm/urdf/arm.urdf (robot description, URDF)
Before this commit: robot arm, 7 links, 6 joints
Links:
- link Baseplate_Part: geometry collision mesh filename=package://curie_robot_description/arm/meshes/Baseplate_Part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; visual mesh filename=package://curie_robot_description/arm/meshes/Baseplate_Part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
- link Bicep_Linkage: geometry collision mesh filename=package://curie_robot_description/arm/meshes/Bicep_Linkage.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; visual mesh filename=package://curie_robot_description/arm/meshes/Bicep_Linkage.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
- link Forearm_Linkage: geometry collision mesh filename=package://curie_robot_description/arm/meshes/Forearm_Linkag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; visual mesh filename=package://curie_robot_description/arm/meshes/Forearm_Linkag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
- link Shoulder: geometry collision mesh filename=package://curie_robot_description/arm/meshes/Shoulder.STL; visual mesh filename=package://curie_robot_description/arm/meshes/Shoulder.STL
- link Wrist_Pitch: geometry collision mesh filename=package://curie_robot_description/arm/meshes/Wrist_Pitch.STL; visual mesh filename=package://curie_robot_description/arm/meshes/Wrist_Pitch.STL
- link Wrist_Roll: geometry collision mesh filename=package://curie_robot_description/arm/meshes/Wrist_Roll.STL; visual mesh filename=package://curie_robot_description/arm/meshes/Wrist_Roll.STL
