Commit message: Rename arm joints and added ros2 controller

File: curie_ws/src/curie_arm_moveit_config/config/arm.ros2_control.xacro (robot description, xacro)
@@ -8,8 +8,8 @@
                 <plugin>mock_components/GenericSystem</plugin>
             </hardware>
-            <joint name="Shoulder_joint">
+            <joint name="Base_joint">
                 <command_interface name="position"/>
                 <state_interface name="position">
-                  <param name="initial_value">${initial_positions['Shoulder_joint']}</param>
+                  <param name="initial_value">${initial_positions['Base_joint']}</param>
                 </state_interface>
                 <state_interface name="velocity"/>
@@ -29,8 +29,8 @@
                 <state_interface name="velocity"/>
             </joint>
-            <joint name="Wrist_roll_joint">
+            <joint name="Wrist_pitch_joint">
                 <command_interface name="position"/>
                 <state_interface name="position">
-                  <param name="initial_value">${initial_positions['Wrist_roll_joint']}</param>
+                  <param name="initial_value">${initial_positions['Wrist_pitch_joint']}</param>
                 </state_interface>
                 <state_interface name="velocity"/>

File: curie_ws/src/curie_robot_description/arm/urdf/arm.urdf (robot description, URDF)
Before this commit: robot arm, 7 links, 6 joints
Links:
- removed link Shoulder
- removed link Wrist_Roll
- added link Base, mass 0.200258048039819; collision mesh filename=package://curie_robot_description/arm/meshes/Shoulder.STL; visual mesh filename=package://curie_robot_description/arm/meshes/Shoulder.STL
- added link Wrist_Base, mass 0.224814880452066; collision mesh filename=package://curie_robot_description/arm/meshes/Wrist_Pitch.STL; visual mesh filename=package://curie_robot_description/arm/meshes/Wrist_Pitch.STL
- link Wrist_Pitch: mass 0.224814880452066 -> 0.160457867162933; geometry collision mesh filename=package://curie_robot_description/arm/meshes/Wrist_Roll.STL; visual mesh filename=package://curie_robot_description/arm/meshes/Wrist_Roll.STL
Joints:
- removed joint Shoulder_joint
- removed joint Wrist_roll_joint
- added joint Base_joint: type continuous, parent Baseplate_Part, child Base, origin xyz=0.0314355367866296 -0.167112129632076 0.0215333450507679 rpy=1.5707963267949 0 0.0124137542544794, axis 0 1 0
- added joint Wrist_base_joint: type fixed, parent Forearm_Linkage, child Wrist_Base, origin xyz=0.0614760326108716 -0.449236652255744 0.0948418360911152 rpy=-2.41679788371581 0.00131623687607705 1.59248518727762, axis 0 0 0
- joint Bicep_Joint: parent Shoulder -> Base
- joint Wrist_pitch_joint: axis 0 0 0 -> 1 0 0; origin xyz=0.0614760326108716 -0.449236652255744 0.0948418360911152 rpy=-2.41679788371581 0.00131623687607705 1.59248518727762 -> xyz=-0.0404563209238247 -0.0124767317892557 0.0124767317892556 rpy=-2.03938401887035 0.785398163397445 -1.57079632679489; parent Forearm_Linkage -> Wrist_Base; type fixed -> continuous

Commit message: Added vcan parameter and regenerated moveit configs

File: curie_ws/src/curie_arm_moveit_config/config/arm.ros2_control.xacro (robot description, xacro)
@@ -1,9 +1,10 @@
 <?xml version="1.0"?>
 <robot xmlns:xacro="http://www.ros.org/wiki/xacro">
-    <xacro:macro name="arm_ros2_control" params="name initial_positions_file">
+    <xacro:macro name="arm_ros2_control" params="name initial_positions_file use_vcan">
         <xacro:property name="initial_positions" value="${load_yaml(initial_positions_file)['initial_positions']}"/>
         <ros2_control name="${name}" type="system">
             <hardware>
                 <plugin>curie_arm_controller/CurieArmController</plugin>
+                <param name="use_vcan">${use_vcan}</param>
             </hardware>
             <joint name="Base_joint">

File: curie_ws/src/curie_arm_moveit_config/config/arm.urdf.xacro (robot description, xacro)
@@ -2,8 +2,9 @@
 <robot xmlns:xacro="http://www.ros.org/wiki/xacro" name="arm">
     <xacro:arg name="initial_positions_file" default="initial_positions.yaml" />
+    <xacro:arg name="use_vcan" default="true" />
     <!-- Import arm urdf file -->
     <xacro:include filename="$(find curie_robot_description)/arm/urdf/arm.urdf" />
     <!-- Import control_xacro -->
     <xacro:include filename="arm.ros2_control.xacro" />
-    <xacro:arm_ros2_control name="FakeSystem" initial_positions_file="$(arg initial_positions_file)"/>
+    <xacro:arm_ros2_control name="ArmSystem" initial_positions_file="$(arg initial_positions_file)" use_vcan="$(arg use_vcan)"/>
 </robot>

File: curie_ws/src/curie_drive_controller/config/mock_diffbot.ros2_control.xacro (robot description, xacro)
@@ -1,17 +1,10 @@
 <?xml version="1.0"?>
 <robot xmlns:xacro="http://www.ros.org/wiki/xacro">
-  <xacro:macro name="mock_diffbot_ros2_control" params="name prefix use_mock_hardware">
+  <xacro:macro name="mock_diffbot_ros2_control" params="name prefix use_vcan">
     <ros2_control name="${name}" type="system">
-      <xacro:unless value="${use_mock_hardware}">
-        <hardware>
-          <plugin>curie_drive_controller/CurieDiffDriveController</plugin>
-        </hardware>
-      </xacro:unless>
-      <xacro:if value="${use_mock_hardware}">
-        <hardware>
-          <plugin>mock_components/GenericSystem</plugin>
-          <param name="calculate_dynamics">true</param>
-        </hardware>
-      </xacro:if>
+      <hardware>
+        <plugin>curie_drive_controller/CurieDiffDriveController</plugin>
+        <param name="use_vcan">${use_vcan}</param>
+      </hardware>
       <joint name="${prefix}front_left_wheel_joint">
         <command_interface name="velocity"/>

File: curie_ws/src/curie_drive_controller/config/mock_diffbot.urdf.xacro (robot description, xacro)
@@ -3,5 +3,5 @@
 <robot xmlns:xacro="http://www.ros.org/wiki/xacro" name="diffdrive_robot">
   <xacro:arg name="prefix" default="" />
-  <xacro:arg name="use_mock_hardware" default="false" />
+  <xacro:arg name="use_vcan" default="true" />
   <xacro:include filename="$(find curie_robot_description)/mock_diffbot/urdf/mock_diffbot_description.urdf.xacro" />
   <!-- Import Rviz colors -->
@@ -11,4 +11,4 @@
   <xacro:diffbot prefix="$(arg prefix)" />
   <xacro:mock_diffbot_ros2_control
-    name="MockDiffBot" prefix="$(arg prefix)" use_mock_hardware="$(arg use_mock_hardware)"/>
+    name="MockDiffBot" prefix="$(arg prefix)" use_vcan="$(arg use_vcan)" />
 </robot>

Commit message: Update arm URDF with gripper

File: curie_ws/src/curie_arm_moveit_config/config/arm.ros2_control.xacro (robot description, xacro)
@@ -8,29 +8,36 @@
                 <param name="use_vcan">${use_vcan}</param>
             </hardware>
-            <joint name="Base_joint">
+            <joint name="base_rotation">
                 <command_interface name="position"/>
                 <state_interface name="position">
-                  <param name="initial_value">${initial_positions['Base_joint']}</param>
+                  <param name="initial_value">${initial_positions['base_rotation']}</param>
                 </state_interface>
                 <state_interface name="velocity"/>
             </joint>
-            <joint name="Bicep_Joint">
+            <joint name="shoulder_joint">
                 <command_interface name="position"/>
                 <state_interface name="position">
-                  <param name="initial_value">${initial_positions['Bicep_Joint']}</param>
+                  <param name="initial_value">${initial_positions['shoulder_joint']}</param>
                 </state_interface>
                 <state_interface name="velocity"/>
             </joint>
-            <joint name="Forearm_Joint">
+            <joint name="elbow_joint">
                 <command_interface name="position"/>
                 <state_interface name="position">
-                  <param name="initial_value">${initial_positions['Forearm_Joint']}</param>
+                  <param name="initial_value">${initial_positions['elbow_joint']}</param>
                 </state_interface>
                 <state_interface name="velocity"/>
             </joint>
-            <joint name="Wrist_pitch_joint">
+            <joint name="wrist_pitch">
                 <command_interface name="position"/>
                 <state_interface name="position">
-                  <param name="initial_value">${initial_positions['Wrist_pitch_joint']}</param>
+                  <param name="initial_value">${initial_positions['wrist_pitch']}</param>
+                </state_interface>
+                <state_interface name="velocity"/>
+            </joint>
+            <joint name="wrist_roll">
+                <command_interface name="position"/>
+                <state_interface name="position">
+                  <param name="initial_value">${initial_positions['wrist_roll']}</param>
                 </state_interface>
                 <state_interface name="velocity"/>

File: curie_ws/src/curie_robot_description/arm/urdf/arm.urdf (robot description, URDF)
Before this commit: robot arm, 7 links, 6 joints
Links:
- removed link Base
- removed link Baseplate_Part
- removed link Bicep_Linkage
- removed link Forearm_Linkage
- removed link Wrist_Base
- removed link Wrist_Pitch
- added link base_link, mass 0.144089467104784; collision mesh filename=package://curie_robot_description/arm/meshes/base_link.STL; visual mesh filename=package://curie_robot_description/arm/meshes/base_link.STL
- added link bicep_Link, mass 0.71055376786355; collision mesh filename=package://curie_robot_description/arm/meshes/bicep_Link.STL; visual mesh filename=package://curie_robot_description/arm/meshes/bicep_Link.STL
- added link endeffector_link, mass 0.288715575983165; collision mesh filename=package://curie_robot_description/arm/meshes/endeffector_li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; visual mesh filename=package://curie_robot_description/arm/meshes/endeffector_li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
- added link forearm_Link, mass 0.443962186668402; collision mesh filename=package://curie_robot_description/arm/meshes/forearm_Link.S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; visual mesh filename=package://curie_robot_description/arm/meshes/forearm_Link.S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
- added link jaw_link, mass 0.0984789337215444; collision mesh filename=package://curie_robot_description/arm/meshes/jaw_link.STL; visual mesh filename=package://curie_robot_description/arm/meshes/jaw_link.STL
- added link shoulder_Link, mass 0.20025804803982; collision mesh filename=package://curie_robot_description/arm/meshes/shoulder_Link.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; visual mesh filename=package://curie_robot_description/arm/meshes/shoulder_Link.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
- added link wrist_link, mass 0.170674141371088; collision mesh filename=package://curie_robot_description/arm/meshes/wrist_link.STL; visual mesh filename=package://curie_robot_description/arm/meshes/wrist_link.STL
Joints:
- removed joint Base_joint
- removed joint Bicep_Joint
- removed joint Forearm_Joint
- removed joint Wrist_base_joint
- removed joint Wrist_pitch_joint
- added joint base_rotation: type continuous, parent base_link, child shoulder_Link, origin xyz=0 0 0 rpy=1.5708 0 0.087908, axis 0 1 0
- added joint elbow_joint: type continuous, parent bicep_Link, child forearm_Link, origin xyz=0.20793 0.43928 0.018326 rpy=-0.081535 0.027551 1.1836, axis 0.060581 0 -0.99816
- added joint gripper: type continuous, parent endeffector_link, child jaw_link, origin xyz=0 -0.0155 -0.085565 rpy=1.5708 0 0, axis 1 0 0
- added joint shoulder_joint: type continuous, parent shoulder_Link, child bicep_Link, origin xyz=0 0.22114 0 rpy=-0.031089 0.0056647 0.36044, axis 0.087795 0 -0.99614
- added joint wrist_pitch: type continuous, parent forearm_Link, child wrist_link, origin xyz=0.049101 -0.49007 0.022058 rpy=-2.3345 -1.5102 -3.1416, axis 1 0 0
- added joint wrist_roll: type continuous, parent wrist_link, child endeffector_link, origin xyz=0.03651 -0.0078577 0.0078577 rpy=-2.3562 0 0, axis 0 0 1
- joint world_to_base: child Baseplate_Part -> base_link

Commit message: Pose planning working somewhat reliably

File: curie_ws/src/curie_arm_moveit_config/config/arm.ros2_control.xacro (robot description, xacro)
@@ -1,11 +1,18 @@
 <?xml version="1.0"?>
 <robot xmlns:xacro="http://www.ros.org/wiki/xacro">
-    <xacro:macro name="arm_ros2_control" params="name initial_positions_file use_vcan">
+    <xacro:macro name="arm_ros2_control" params="name initial_positions_file use_vcan use_mock_hardware">
         <xacro:property name="initial_positions" value="${load_yaml(initial_positions_file)['initial_positions']}"/>
         <ros2_control name="${name}" type="system">
-            <hardware>
-                <plugin>curie_arm_controller/CurieArmController</plugin>
-                <param name="use_vcan">${use_vcan}</param>
-            </hardware>
+            <xacro:if value="${use_mock_hardware}">
+                <hardware>
+                    <plugin>mock_components/GenericSystem</plugin>
+                </hardware>
+            </xacro:if>
+            <xacro:unless value="${use_mock_hardware}">
+                <hardware>
+                    <plugin>curie_arm_controller/CurieArmController</plugin>
+                    <param name="use_vcan">${use_vcan}</param>
+                </hardware>
+            </xacro:unless>
             <joint name="base_rotation">
                 <command_interface name="position"/>

File: curie_ws/src/curie_arm_moveit_config/config/arm.urdf.xacro (robot description, xacro)
@@ -3,8 +3,9 @@
     <xacro:arg name="initial_positions_file" default="initial_positions.yaml" />
     <xacro:arg name="use_vcan" default="false" />
+    <xacro:arg name="use_mock_hardware" default="true" />
     <!-- Import arm urdf file -->
     <xacro:include filename="$(find curie_robot_description)/arm/urdf/arm.urdf" />
     <!-- Import control_xacro -->
     <xacro:include filename="arm.ros2_control.xacro" />
-    <xacro:arm_ros2_control name="ArmSystem" initial_positions_file="$(arg initial_positions_file)" use_vcan="$(arg use_vcan)"/>
+    <xacro:arm_ros2_control name="ArmSystem" initial_positions_file="$(arg initial_positions_file)" use_vcan="$(arg use_vcan)" use_mock_hardware="$(arg use_mock_hardware)"/>
 </robot>

File: curie_ws/src/curie_robot_description/arm/urdf/arm.urdf (robot description, URDF)
Before this commit: robot arm, 8 links, 7 joints
Joints:
- joint base_rotation: limit (none) -> lower=-2.35 upper=2.35 effort=5 velocity=5; type continuous -> revolute
- joint elbow_joint: limit (none) -> lower=-0.79 upper=1.57 effort=5 velocity=5; type continuous -> revolute
- joint gripper: limit (none) -> lower=0 upper=1.57 effort=5 velocity=5; type continuous -> revolute
- joint shoulder_joint: limit (none) -> lower=-1.57 upper=1.57 effort=5 velocity=5; type continuous -> revolute
- joint wrist_pitch: limit (none) -> lower=-1.57 upper=1.57 effort=5 velocity=5; type continuous -> revolute
- joint wrist_roll: limit (none) -> lower=-1.57 upper=1.57 effort=5 velocity=5; type continuous -> revolute

Commit message: Add gripper joint, resolve issue 53

File: curie_ws/src/curie_arm_moveit_config/config/arm.ros2_control.xacro (robot description, xacro)
@@ -50,4 +50,11 @@
                 <state_interface name="velocity"/>
             </joint>
+            <joint name="gripper_joint">
+                <command_interface name="position"/>
+                <state_interface name="position">
+                  <param name="initial_value">0.0</param> <!-- {initial_positions['gripper_joint']} -->
+                </state_interface>
+                <state_interface name="velocity"/>
+            </joint>
         </ros2_control>
     </xacro:macro>
