Commit message: Integrated sparkmax mocking

File: curie_ws/src/curie_arm_moveit_config/config/arm.ros2_control.xacro (robot description, xacro)
@@ -1,18 +1,11 @@
 <?xml version="1.0"?>
 <robot xmlns:xacro="http://www.ros.org/wiki/xacro">
-    <xacro:macro name="arm_ros2_control" params="name initial_positions_file use_vcan use_mock_hardware">
+    <xacro:macro name="arm_ros2_control" params="name initial_positions_file use_mock_hardware">
         <xacro:property name="initial_positions" value="${load_yaml(initial_positions_file)['initial_positions']}"/>
         <ros2_control name="${name}" type="system">
-            <xacro:if value="${use_mock_hardware}">
-                <hardware>
-                    <plugin>mock_components/GenericSystem</plugin>
-                </hardware>
-            </xacro:if>
-            <xacro:unless value="${use_mock_hardware}">
-                <hardware>
-                    <plugin>curie_arm_controller/CurieArmController</plugin>
-                    <param name="use_vcan">${use_vcan}</param>
-                </hardware>
-            </xacro:unless>
+            <hardware>
+                <plugin>curie_arm_controller/CurieArmController</plugin>
+                <param name="use_vcan">${use_mock_hardware}</param>
+            </hardware>
             <joint name="base_rotation">
                 <command_interface name="position"/>

File: curie_ws/src/curie_arm_moveit_config/config/arm.urdf.xacro (robot description, xacro)
@@ -2,5 +2,4 @@
 <robot xmlns:xacro="http://www.ros.org/wiki/xacro" name="arm">
     <xacro:arg name="initial_positions_file" default="initial_positions.yaml" />
-    <xacro:arg name="use_vcan" default="false" />
     <xacro:arg name="use_mock_hardware" default="true" />
     <!-- Import arm urdf file -->
@@ -8,4 +7,4 @@
     <!-- Import control_xacro -->
     <xacro:include filename="arm.ros2_control.xacro" />
-    <xacro:arm_ros2_control name="ArmSystem" initial_positions_file="$(arg initial_positions_file)" use_vcan="$(arg use_vcan)" use_mock_hardware="$(arg use_mock_hardware)"/>
+    <xacro:arm_ros2_control name="ArmSystem" initial_positions_file="$(arg initial_positions_file)" use_mock_hardware="$(arg use_mock_hardware)"/>
 </robot>

File: curie_ws/src/curie_drive_controller/config/mock_diffbot.ros2_control.xacro (robot description, xacro)
@@ -1,9 +1,9 @@
 <?xml version="1.0"?>
 <robot xmlns:xacro="http://www.ros.org/wiki/xacro">
-  <xacro:macro name="mock_diffbot_ros2_control" params="name prefix use_vcan">
+  <xacro:macro name="mock_diffbot_ros2_control" params="name prefix use_mock_hardware">
     <ros2_control name="${name}" type="system">
       <hardware>
         <plugin>curie_drive_controller/CurieDiffDriveController</plugin>
-        <param name="use_vcan">${use_vcan}</param>
+        <param name="use_vcan">${use_mock_hardware}</param>
       </hardware>
       <joint name="${prefix}front_left_wheel_joint">

File: curie_ws/src/curie_drive_controller/config/mock_diffbot.urdf.xacro (robot description, xacro)
@@ -3,5 +3,5 @@
 <robot xmlns:xacro="http://www.ros.org/wiki/xacro" name="diffdrive_robot">
   <xacro:arg name="prefix" default="" />
-  <xacro:arg name="use_vcan" default="true" />
+  <xacro:arg name="use_mock_hardware" default="true" />
   <xacro:include filename="$(find curie_robot_description)/mock_diffbot/urdf/mock_diffbot_description.urdf.xacro" />
   <!-- Import Rviz colors -->
@@ -11,4 +11,4 @@
   <xacro:diffbot prefix="$(arg prefix)" />
   <xacro:mock_diffbot_ros2_control
-    name="MockDiffBot" prefix="$(arg prefix)" use_vcan="$(arg use_vcan)" />
+    name="MockDiffBot" prefix="$(arg prefix)" use_vcan="$(arg use_mock_hardware)" />
 </robot>

Commit message: Merge main into feature/hand

File: curie_ws/src/curie_arm_moveit_config/config/arm.ros2_control.xacro (robot description, xacro)
@@ -1,20 +1,15 @@
 <?xml version="1.0"?>
 <robot xmlns:xacro="http://www.ros.org/wiki/xacro">
-    <xacro:macro name="arm_ros2_control" params="name initial_positions_file use_vcan use_mock_hardware">
+    <xacro:macro name="arm_ros2_control" params="name initial_positions_file use_mock_hardware">
         <xacro:property name="initial_positions" value="${load_yaml(initial_positions_file)['initial_positions']}"/>
         <ros2_control name="${name}" type="system">
-            <xacro:if value="${use_mock_hardware}">
-                <hardware>
-                    <plugin>mock_components/GenericSystem</plugin>
-                </hardware>
-            </xacro:if>
-            <xacro:unless value="${use_mock_hardware}">
-                <hardware>
-                    <plugin>curie_arm_controller/CurieArmController</plugin>
-                    <param name="use_vcan">${use_vcan}</param>
-                </hardware>
-            </xacro:unless>
+            <hardware>
+                <plugin>curie_arm_controller/CurieArmController</plugin>
+                <param name="use_vcan">${use_mock_hardware}</param>
+                <!-- <plugin>mock_components/GenericSystem</plugin> -->
+            </hardware>
             <joint name="base_rotation">
                 <command_interface name="position"/>
+                <command_interface name="velocity"/>
                 <state_interface name="position">
                   <param name="initial_value">${initial_positions['base_rotation']}</param>
@@ -24,4 +19,5 @@
             <joint name="shoulder_joint">
                 <command_interface name="position"/>
+                <command_interface name="velocity"/>
                 <state_interface name="position">
                   <param name="initial_value">${initial_positions['shoulder_joint']}</param>
@@ -31,4 +27,5 @@
             <joint name="elbow_joint">
                 <command_interface name="position"/>
+                <command_interface name="velocity"/>
                 <state_interface name="position">
                   <param name="initial_value">${initial_positions['elbow_joint']}</param>
@@ -38,4 +35,5 @@
             <joint name="wrist_pitch">
                 <command_interface name="position"/>
+                <command_interface name="velocity"/>
                 <state_interface name="position">
                   <param name="initial_value">${initial_positions['wrist_pitch']}</param>
@@ -45,4 +43,5 @@
             <joint name="wrist_roll">
                 <command_interface name="position"/>
+                <command_interface name="velocity"/>
                 <state_interface name="position">
                   <param name="initial_value">${initial_positions['wrist_roll']}</param>

Commit message: Rename gripper joint

File: curie_ws/src/curie_arm_moveit_config/config/arm.ros2_control.xacro (robot description, xacro)
@@ -49,5 +49,5 @@
                 <state_interface name="velocity"/>
             </joint>
-            <joint name="gripper_joint">
+            <joint name="gripper">
                 <command_interface name="position"/>
                 <state_interface name="position">

Commit message: add low-pass filter for curie_arm

File: curie_ws/src/curie_arm_moveit_config/config/arm.ros2_control.xacro (robot description, xacro)
@@ -2,9 +2,15 @@
 <robot xmlns:xacro="http://www.ros.org/wiki/xacro">
     <xacro:macro name="arm_ros2_control" params="name initial_positions_file use_mock_hardware">
-        <xacro:property name="initial_positions" value="${load_yaml(initial_positions_file)['initial_positions']}"/>
+        <xacro:property
+            name="initial_positions"
+            value="${load_yaml(initial_positions_file)['initial_positions']}"/>
         <ros2_control name="${name}" type="system">
             <hardware>
                 <plugin>curie_arm_controller/CurieArmController</plugin>
                 <param name="use_vcan">${use_mock_hardware}</param>
+                <param name="lpf_sampling_frequency">50.0</param>
+                <!-- placeholder for damping parameters -->
+                <param name="lpf_damping_frequency">5.0</param>
+                <param name="lpf_damping_intensity">0.0</param>
                 <!-- <plugin>mock_components/GenericSystem</plugin> -->
             </hardware>
@@ -13,7 +19,8 @@
                 <command_interface name="velocity"/>
                 <state_interface name="position">
-                  <param name="initial_value">${initial_positions['base_rotation']}</param>
+                    <param name="initial_value">${initial_positions['base_rotation']}</param>
                 </state_interface>
                 <state_interface name="velocity"/>
+                <state_interface name="raw_position"/>
             </joint>
             <joint name="shoulder_joint">
@@ -21,7 +28,8 @@
                 <command_interface name="velocity"/>
                 <state_interface name="position">
-                  <param name="initial_value">${initial_positions['shoulder_joint']}</param>
+                    <param name="initial_value">${initial_positions['shoulder_joint']}</param>
                 </state_interface>
                 <state_interface name="velocity"/>
+                <state_interface name="raw_position"/>
             </joint>
             <joint name="elbow_joint">
@@ -29,7 +37,8 @@
                 <command_interface name="velocity"/>
                 <state_interface name="position">
-                  <param name="initial_value">${initial_positions['elbow_joint']}</param>
+                    <param name="initial_value">${initial_positions['elbow_joint']}</param>
                 </state_interface>
                 <state_interface name="velocity"/>
+                <state_interface name="raw_position"/>
             </joint>
             <joint name="wrist_pitch">
@@ -37,7 +46,8 @@
                 <command_interface name="velocity"/>
                 <state_interface name="position">
-                  <param name="initial_value">${initial_positions['wrist_pitch']}</param>
+                    <param name="initial_value">${initial_positions['wrist_pitch']}</param>
                 </state_interface>
                 <state_interface name="velocity"/>
+                <state_interface name="raw_position"/>
             </joint>
             <joint name="wrist_roll">
@@ -45,14 +55,16 @@
                 <command_interface name="velocity"/>
                 <state_interface name="position">
-                  <param name="initial_value">${initial_positions['wrist_roll']}</param>
+                    <param name="initial_value">${initial_positions['wrist_roll']}</param>
                 </state_interface>
                 <state_interface name="velocity"/>
+                <state_interface name="raw_position"/>
             </joint>
             <joint name="gripper">
                 <command_interface name="position"/>
                 <state_interface name="position">
-                  <param name="initial_value">${initial_positions['gripper']}</param>
+                    <param name="initial_value">${initial_positions['gripper']}</param>
                 </state_interface>
                 <state_interface name="velocity"/>
+                <state_interface name="raw_position"/>
             </joint>
         </ros2_control>
