Commit message: Invert bicep joint direction

File: curie_ws/src/curie_robot_description/arm/urdf/arm.urdf (robot description, URDF)
Before this commit: robot arm, 7 links, 6 joints
Joints:
- joint Bicep_Joint: axis 0.0877948496902314 0 -0.996138576889716 -> 0 0 1
- joint Forearm_Joint: axis 0.0605805514570394 0 -0.998163311680589 -> 0 0 -1
