Commit message: revolute joints

File: curie_ws/src/curie_robot_description/arm/urdf/arm.urdf (robot description, URDF)
Before this commit: robot arm, 7 links, 6 joints
Joints:
- joint Base_joint: limit (none) -> lower=-3.14 upper=3.14 effort=10 velocity=5.0; type continuous -> revolute
- joint Bicep_Joint: limit (none) -> lower=-1.57 upper=1.57 effort=10 velocity=5.0; type continuous -> revolute
- joint Forearm_Joint: limit (none) -> lower=-1.57 upper=1.57 effort=10 velocity=5.0; type continuous -> revolute
- joint Wrist_pitch_joint: limit (none) -> lower=-1.57 upper=1.57 effort=10 velocity=5.0; type continuous -> revolute
